File: Esquemas de ligação/dispositivos-i2c.sch (EAGLE design)
At the start: 6 parts

Commit message: Esquemático - Dispositivos I2C
Connections:
- removed net N$1: ESP-8266.VIN
- removed net N$2: ESP-8266.GND@2
- net GND: now also ESP-8266.GND@2
- net VCC: now also ESP-8266.VIN
Changed lines of the file:
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@@
 </busses>
 <nets>
-<net name="N$1" class="0">
-<segment>
-<pinref part="ESP-8266" gate="G$1" pin="VIN"/>
-<wire x1="2.54" y1="38.1" x2="-7.62" y2="38.1" width="0.1524" layer="91"/>
-<label x="-7.62" y="38.1" size="1.778" layer="95" rot="R180" xref="yes"/>
-</segment>
-</net>
-<net name="N$2" class="0">
-<segment>
-<pinref part="ESP-8266" gate="G$1" pin="GND@2"/>
-<wire x1="2.54" y1="40.64" x2="0" y2="40.64" width="0.1524" layer="91"/>
-<label x="0" y="40.64" size="1.778" layer="95" rot="R180" xref="yes"/>
-</segment>
-</net>
 <net name="GND" class="0">
 <segment>
@@
 <junction x="81.28" y="-27.94"/>
 </segment>
+<segment>
+<pinref part="ESP-8266" gate="G$1" pin="GND@2"/>
+<wire x1="2.54" y1="40.64" x2="0" y2="40.64" width="0.1524" layer="91"/>
+<label x="0" y="40.64" size="1.778" layer="95" rot="R180" xref="yes"/>
+</segment>
 </net>
 <net name="VCC" class="0">
@@
 <wire x1="86.36" y1="-22.86" x2="86.36" y2="-17.78" width="0.1524" layer="91"/>
 </segment>
+<segment>
+<pinref part="ESP-8266" gate="G$1" pin="VIN"/>
+<wire x1="2.54" y1="38.1" x2="-7.62" y2="38.1" width="0.1524" layer="91"/>
+<label x="-7.62" y="38.1" size="1.778" layer="95" rot="R180" xref="yes"/>
+</segment>
 </net>
