File: Projeto final/Projeto Final.brd (EAGLE design)
At the start: 60.9 x 63.5 mm, 6 parts

Commit message: Arquivos projeto final
Parts:
- removed LIMITADOR-TENSAO: 7805L, linear:TO92
- added IC1: (no value), v-reg:78XXL
Connections:
- net GND: now also IC1.GND; no longer LIMITADOR-TENSAO.2
- net IN_12V: now also IC1.IN; no longer LIMITADOR-TENSAO.3
- net VIN_ESP: now also IC1.OUT; no longer LIMITADOR-TENSAO.1
Routing:
- net VIN_ESP: track 130.1 -> 147.5 mm
- net GND: track 106.2 -> 114.7 mm
- net IN_12V: track 21.9 -> 26.2 mm
Changed lines of the file:
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@@
 <layer number="14" name="Route14" color="1" fill="6" visible="no" active="no"/>
 <layer number="15" name="Route15" color="4" fill="6" visible="no" active="no"/>
-<layer number="16" name="Bottom" color="1" fill="1" visible="no" active="yes"/>
+<layer number="16" name="Bottom" color="1" fill="1" visible="yes" active="yes"/>
 <layer number="17" name="Pads" color="2" fill="1" visible="yes" active="yes"/>
 <layer number="18" name="Vias" color="2" fill="1" visible="yes" active="yes"/>
@@
 <layer number="20" name="Dimension" color="24" fill="1" visible="yes" active="yes"/>
 <layer number="21" name="tPlace" color="7" fill="1" visible="yes" active="yes"/>
-<layer number="22" name="bPlace" color="7" fill="1" visible="no" active="yes"/>
+<layer number="22" name="bPlace" color="7" fill="1" visible="yes" active="yes"/>
 <layer number="23" name="tOrigins" color="15" fill="1" visible="yes" active="yes"/>
-<layer number="24" name="bOrigins" color="15" fill="1" visible="no" active="yes"/>
+<layer number="24" name="bOrigins" color="15" fill="1" visible="yes" active="yes"/>
 <layer number="25" name="tNames" color="7" fill="1" visible="yes" active="yes"/>
-<layer number="26" name="bNames" color="7" fill="1" visible="no" active="yes"/>
+<layer number="26" name="bNames" color="7" fill="1" visible="yes" active="yes"/>
 <layer number="27" name="tValues" color="7" fill="1" visible="no" active="yes"/>
 <layer number="28" name="bValues" color="7" fill="1" visible="no" active="yes"/>
@@
 <layer number="38" name="bTest" color="7" fill="1" visible="no" active="yes"/>
 <layer number="39" name="tKeepout" color="4" fill="11" visible="yes" active="yes"/>
-<layer number="40" name="bKeepout" color="1" fill="11" visible="no" active="yes"/>
+<layer number="40" name="bKeepout" color="1" fill="11" visible="yes" active="yes"/>
 <layer number="41" name="tRestrict" color="4" fill="10" visible="yes" active="yes"/>
-<layer number="42" name="bRestrict" color="1" fill="10" visible="no" active="yes"/>
+<layer number="42" name="bRestrict" color="1" fill="10" visible="yes" active="yes"/>
 <layer number="43" name="vRestrict" color="2" fill="10" visible="no" active="yes"/>
 <layer number="44" name="Drills" color="7" fill="1" visible="no" active="yes"/>
@@
 <layer number="49" name="Reference" color="7" fill="1" visible="no" active="yes"/>
 <layer number="51" name="tDocu" color="7" fill="1" visible="yes" active="yes"/>
-<layer number="52" name="bDocu" color="7" fill="1" visible="no" active="yes"/>
+<layer number="52" name="bDocu" color="7" fill="1" visible="yes" active="yes"/>
 <layer number="88" name="SimResults" color="9" fill="1" visible="no" active="no"/>
 <layer number="89" name="SimProbes" color="9" fill="1" visible="no" active="no"/>
@@
 <attribute name="VALUE" x="-4.1656" y="26.4668" size="1.016" layer="27" ratio="10" rot="R270"/>
 </element>
-<element name="LIMITADOR-TENSAO" library="linear" library_urn="urn:adsk.eagle:library:262" package="TO92" package3d_urn="urn:adsk.eagle:package:16416/2" value="7805L" x="0.381" y="44.3738" smashed="yes">
-<attribute name="NAME" x="2.794" y="46.0248" size="1.27" layer="25" ratio="10"/>
-<attribute name="VALUE" x="3.302" y="43.1038" size="1.27" layer="27" ratio="10"/>
-</element>
 <element name="H" library="con-molex" library_urn="urn:adsk.eagle:library:165" package="22-23-2021" value="22-23-2021" x="0.9398" y="34.0614" smashed="yes" rot="R270">
 <attribute name="MF" value="MOLEX" x="11.811" y="40.0812" size="1.778" layer="27" rot="R270" display="off"/>
@@
 <attribute name="VALUE" x="25.8064" y="23.0124" size="1.778" layer="27" rot="R90"/>
 </element>
+<element name="IC1" library="v-reg" library_urn="urn:adsk.eagle:library:409" package="78XXL" package3d_urn="urn:adsk.eagle:package:30361/1" value="" x="0.8636" y="51.181"/>
 </elements>
 <signals>
@@
 <signal name="GND" class="2">
 <contactref element="HCSR-04" pad="1"/>
-<contactref element="LIMITADOR-TENSAO" pad="2"/>
 <contactref element="U$1" pad="GND@2"/>
-<wire x1="0.381" y1="46.2788" x2="0.5762" y2="46.3841" width="2" layer="16"/>
 <wire x1="25.4762" y1="71.7296" x2="24.892" y2="71.1454" width="2" layer="16"/>
 <wire x1="24.892" y1="71.1454" x2="24.892" y2="45.593" width="2" layer="16"/>
@@
 <wire x1="25.7048" y1="44.7294" x2="25.8318" y2="44.6024" width="2" layer="16"/>
 <wire x1="25.8318" y1="44.6024" x2="33.4264" y2="44.6024" width="2" layer="16"/>
-<wire x1="0.5762" y1="46.3841" x2="0.5762" y2="63.0348" width="2" layer="16"/>
-<wire x1="0.5762" y1="63.0348" x2="9.271" y2="71.7296" width="2" layer="16"/>
 <wire x1="9.271" y1="71.7296" x2="25.4762" y2="71.7296" width="2" layer="16"/>
 <wire x1="40.9956" y1="67.5132" x2="40.9956" y2="59.3344" width="2" layer="16"/>
@@
 <wire x1="36.769809375" y1="71.738990625" x2="40.9956" y2="67.5132" width="2" layer="16"/>
 <wire x1="25.4762" y1="71.7296" x2="25.485590625" y2="71.738990625" width="2" layer="16"/>
+<contactref element="IC1" pad="GND"/>
+<wire x1="0.8636" y1="47.371" x2="0.8636" y2="44.1452" width="2" layer="16"/>
+<wire x1="0.8636" y1="44.1452" x2="1.7272" y2="43.2816" width="2" layer="16"/>
+<wire x1="1.7272" y1="43.2816" x2="4.4958" y2="43.2816" width="2" layer="16"/>
+<wire x1="4.4958" y1="43.2816" x2="7.493" y2="46.2788" width="2" layer="16"/>
+<wire x1="7.493" y1="69.9516" x2="9.271" y2="71.7296" width="2" layer="16"/>
+<wire x1="7.493" y1="46.2788" x2="7.493" y2="69.9516" width="2" layer="16"/>
 </signal>
 <signal name="EN_A">
@@
 </signal>
 <signal name="VIN_ESP">
-<contactref element="LIMITADOR-TENSAO" pad="1"/>
 <contactref element="U$1" pad="VIN"/>
-<wire x1="-1.1524" y1="36.0125" x2="-1.1524" y2="44.3674" width="1" layer="16"/>
 <wire x1="-3.5581" y1="33.6068" x2="-1.1524" y2="36.0125" width="1" layer="16"/>
 <wire x1="-3.5581" y1="23.3615" x2="-3.5581" y2="33.6068" width="1" layer="16"/>
@@
 <wire x1="10.3716" y1="24.2004" x2="10.5664" y2="24.2824" width="1" layer="16"/>
 <contactref element="HCSR-04" pad="4"/>
-<wire x1="-0.889" y1="44.3738" x2="-2.6416" y2="46.1264" width="1" layer="16"/>
-<wire x1="-2.6416" y1="46.1264" x2="-2.6416" y2="65.786" width="1" layer="16"/>
-<wire x1="-2.6416" y1="65.786" x2="6.1722" y2="74.5998" width="1" layer="16"/>
-<wire x1="6.1722" y1="74.5998" x2="44.2214" y2="74.5998" width="1" layer="16"/>
 <wire x1="44.2214" y1="74.5998" x2="49.5808" y2="69.2404" width="1" layer="16"/>
 <wire x1="49.5808" y1="69.2404" x2="49.5808" y2="60.2996" width="1" layer="16"/>
 <wire x1="49.5808" y1="60.2996" x2="48.6156" y2="59.3344" width="1" layer="16"/>
-<wire x1="-1.1524" y1="44.3674" x2="-0.889" y2="44.3738" width="0" layer="19" extent="16-16"/>
+<contactref element="IC1" pad="OUT"/>
+<wire x1="-1.1524" y1="36.0125" x2="-1.1524" y2="38.0586" width="1" layer="16"/>
+<wire x1="1.6002" y1="53.34" x2="3.7084" y2="51.2318" width="1" layer="16"/>
+<wire x1="3.7084" y1="51.2318" x2="3.7084" y2="47.6758" width="1" layer="16"/>
+<wire x1="3.7084" y1="47.6758" x2="3.4036" y2="47.371" width="1" layer="16"/>
+<wire x1="-1.1524" y1="38.0586" x2="-4.1148" y2="41.021" width="1" layer="16"/>
+<wire x1="-4.1148" y1="41.021" x2="-4.1148" y2="52.1462" width="1" layer="16"/>
+<wire x1="-4.1148" y1="52.1462" x2="-2.921" y2="53.34" width="1" layer="16"/>
+<wire x1="-2.921" y1="53.34" x2="1.6002" y2="53.34" width="1" layer="16"/>
+<wire x1="1.6002" y1="53.34" x2="-3.0226" y2="57.9628" width="1" layer="16"/>
+<wire x1="-3.0226" y1="57.9628" x2="-3.429" y2="57.9628" width="1" layer="16"/>
+<wire x1="-3.429" y1="57.9628" x2="-4.699" y2="59.2328" width="1" layer="16"/>
+<wire x1="-4.699" y1="59.2328" x2="-4.699" y2="65.8876" width="1" layer="16"/>
+<wire x1="-4.699" y1="65.8876" x2="4.0132" y2="74.5998" width="1" layer="16"/>
+<wire x1="4.0132" y1="74.5998" x2="44.2214" y2="74.5998" width="1" layer="16"/>
 </signal>
 <signal name="IN_12V">
 <contactref element="PIN" pad="1"/>
-<contactref element="LIMITADOR-TENSAO" pad="3"/>
 <contactref element="H" pad="1"/>
-<wire x1="1.4405" y1="35.7244" x2="1.4405" y2="44.3674" width="1" layer="16"/>
 <wire x1="1.1524" y1="35.4363" x2="1.4405" y2="35.7244" width="1" layer="16"/>
-<wire x1="1.4405" y1="44.3674" x2="1.651" y2="44.3738" width="1" layer="16"/>
 <wire x1="1.1524" y1="35.4363" x2="0.9398" y2="35.3314" width="1" layer="16"/>
 <wire x1="0.8643" y1="29.9624" x2="0.8643" y2="25.3528" width="1" layer="16"/>
@@
 <wire x1="0.8643" y1="25.3528" x2="0.9144" y2="25.1968" width="1" layer="16"/>
 <wire x1="0.5762" y1="35.4363" x2="0.9398" y2="35.3314" width="1" layer="16"/>
+<contactref element="IC1" pad="IN"/>
+<wire x1="-1.6764" y1="47.371" x2="-1.6764" y2="43.0022" width="1" layer="16"/>
+<wire x1="1.1524" y1="40.1734" x2="1.1524" y2="35.4363" width="1" layer="16"/>
+<wire x1="-1.6764" y1="43.0022" x2="1.1524" y2="40.1734" width="1" layer="16"/>
 </signal>
 <signal name="IN_GND">
