File: Projeto final/Projeto Final.sch (EAGLE design)
At the start: 6 parts

Commit message: Arquivos projeto final
Parts:
- removed LIMITADOR-TENSAO: 7805L, linear:7805L
- added IC1: (no value), v-reg:78XXL
Connections:
- net GND: now also IC1.GND; no longer LIMITADOR-TENSAO.GND
- net IN_12V: now also IC1.IN; no longer LIMITADOR-TENSAO.VI
- net VIN_ESP: now also IC1.OUT; no longer LIMITADOR-TENSAO.VO
Changed lines of the file:
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@@
 <part name="PONTE_H" library="con-lstb" library_urn="urn:adsk.eagle:library:162" deviceset="MA06-1" device="" package3d_urn="urn:adsk.eagle:package:8340/1"/>
 <part name="PIN" library="con-molex" library_urn="urn:adsk.eagle:library:165" deviceset="22-23-2021" device=""/>
-<part name="LIMITADOR-TENSAO" library="linear" library_urn="urn:adsk.eagle:library:262" deviceset="78*" device="L" package3d_urn="urn:adsk.eagle:package:16416/2" technology="05"/>
 <part name="H" library="con-molex" library_urn="urn:adsk.eagle:library:165" deviceset="22-23-2021" device=""/>
 <part name="U$1" library="ESP12E_DEVKIT" deviceset="ESP12E_DEVKIT" device=""/>
 <part name="FRAME1" library="frames" deviceset="A4L-LOC" device=""/>
+<part name="IC1" library="v-reg" library_urn="urn:adsk.eagle:library:409" deviceset="78XXL" device="" package3d_urn="urn:adsk.eagle:package:30361/1"/>
 </parts>
 <sheets>
@@
 <attribute name="NAME" x="93.98" y="6.858" size="1.524" layer="95"/>
 </instance>
-<instance part="LIMITADOR-TENSAO" gate="A1" x="127" y="-40.64" smashed="yes">
-<attribute name="NAME" x="119.38" y="-34.925" size="1.778" layer="95"/>
-<attribute name="VALUE" x="119.38" y="-37.465" size="1.778" layer="96"/>
-</instance>
 <instance part="H" gate="-1" x="93.98" y="2.54" smashed="yes">
 <attribute name="NAME" x="96.52" y="1.778" size="1.524" layer="95"/>
@@
 </instance>
 <instance part="FRAME1" gate="G$1" x="22.86" y="-83.82"/>
+<instance part="IC1" gate="A" x="190.5" y="-38.1"/>
 </instances>
 <busses>
@@
 </segment>
 <segment>
-<pinref part="LIMITADOR-TENSAO" gate="A1" pin="GND"/>
-<wire x1="127" y1="-48.26" x2="127" y2="-50.8" width="0.1524" layer="91"/>
-<label x="127" y="-50.8" size="1.778" layer="95" rot="R270" xref="yes"/>
-</segment>
-<segment>
 <pinref part="U$1" gate="G$1" pin="GND@2"/>
 <wire x1="88.9" y1="58.42" x2="93.98" y2="58.42" width="0.1524" layer="91"/>
 <label x="93.98" y="58.42" size="1.778" layer="95" xref="yes"/>
 </segment>
+<segment>
+<pinref part="IC1" gate="A" pin="GND"/>
+<wire x1="190.5" y1="-45.72" x2="190.5" y2="-50.8" width="0.1524" layer="91"/>
+<label x="190.5" y="-50.8" size="1.778" layer="95" xref="yes"/>
+</segment>
 </net>
 <net name="EN_A" class="0">
@@
 </net>
 <net name="VIN_ESP" class="0">
-<segment>
-<pinref part="LIMITADOR-TENSAO" gate="A1" pin="VO"/>
-<wire x1="137.16" y1="-40.64" x2="149.86" y2="-40.64" width="0.1524" layer="91"/>
-<label x="149.86" y="-40.64" size="1.778" layer="95" xref="yes"/>
-</segment>
 <segment>
 <pinref part="U$1" gate="G$1" pin="VIN"/>
@@
 <label x="200.66" y="40.64" size="1.778" layer="95" xref="yes"/>
 </segment>
+<segment>
+<pinref part="IC1" gate="A" pin="OUT"/>
+<wire x1="198.12" y1="-38.1" x2="203.2" y2="-38.1" width="0.1524" layer="91"/>
+<label x="203.2" y="-38.1" size="1.778" layer="95" xref="yes"/>
+</segment>
 </net>
 <net name="IN_12V" class="0">
@@
 </segment>
 <segment>
-<pinref part="LIMITADOR-TENSAO" gate="A1" pin="VI"/>
-<wire x1="116.84" y1="-40.64" x2="114.3" y2="-40.64" width="0.1524" layer="91"/>
-<label x="114.3" y="-40.64" size="1.778" layer="95" rot="R180" xref="yes"/>
-</segment>
-<segment>
 <pinref part="H" gate="-1" pin="S"/>
 <wire x1="91.44" y1="2.54" x2="83.82" y2="2.54" width="0.1524" layer="91"/>
 <label x="83.82" y="2.54" size="1.778" layer="95" rot="R180" xref="yes"/>
 </segment>
-</net>
+<segment>
+<pinref part="IC1" gate="A" pin="IN"/>
+<wire x1="182.88" y1="-38.1" x2="177.8" y2="-38.1" width="0.1524" layer="91"/>
+<label x="177.8" y="-38.1" size="1.778" layer="95" xref="yes"/>
+</segment>
+</net>
